File: Raspberry_PI_Board/Raspberry_PI_Board.kicad_sch (KiCad schematic)
At the start: 3 parts, among them J1 Conn_02x08_Odd_Even, J2 Conn_02x08_Odd_Even, U3 RASPBERRY_PI_ZERO_2_W

Commit message: Fix flipped components
Connections:
- net Passthrough_Voltage is gone; now on net +5V: J1.1 (Pin_1), J1.11 (Pin_11), J1.13 (Pin_13), J1.15 (Pin_15), J1.3 (Pin_3), J1.5 (Pin_5), J1.7 (Pin_7), J1.9 (Pin_9)
